Commit message: G1 stable stance

File: humanoid-legged-description/urdf/humanoid_legged_control.urdf (robot description, URDF)
Before this commit: robot g1_description, 32 links, 31 joints
Joints:
- joint head_joint: origin xyz=0.0039635 0 0.30 rpy=0 0 0 -> xyz=0.0039635 0 -0.044 rpy=0 0 0
- joint left_ankle_pitch_joint: limit lower=-0.87267 upper=0.5236 effort=50 velocity=30 -> lower=-0.87267 upper=0.5236 effort=120 velocity=30
- joint left_ankle_roll_joint: limit lower=-0.2618 upper=0.2618 effort=50 velocity=30 -> lower=-0.2618 upper=0.2618 effort=120 velocity=30
- joint left_hip_pitch_joint: limit lower=-2.5307 upper=2.8798 effort=88 velocity=32 -> lower=-2.5307 upper=2.8798 effort=200 velocity=32
- joint left_hip_roll_joint: limit lower=-0.5236 upper=2.9671 effort=88 velocity=32 -> lower=-0.5236 upper=2.9671 effort=200 velocity=32
- joint left_hip_yaw_joint: limit lower=-2.7576 upper=2.7576 effort=88 velocity=32 -> lower=-2.7576 upper=2.7576 effort=200 velocity=32
- joint left_knee_joint: limit lower=-0.087267 upper=2.8798 effort=139 velocity=20 -> lower=-0.087267 upper=2.8798 effort=250 velocity=20
- joint right_ankle_pitch_joint: limit lower=-0.87267 upper=0.5236 effort=50 velocity=30 -> lower=-0.87267 upper=0.5236 effort=120 velocity=30
- joint right_ankle_roll_joint: limit lower=-0.2618 upper=0.2618 effort=50 velocity=30 -> lower=-0.2618 upper=0.2618 effort=120 velocity=30
- joint right_hip_pitch_joint: limit lower=-2.5307 upper=2.8798 effort=88 velocity=32 -> lower=-2.5307 upper=2.8798 effort=200 velocity=32
- joint right_hip_roll_joint: limit lower=-2.9671 upper=0.5236 effort=88 velocity=32 -> lower=-2.9671 upper=0.5236 effort=200 velocity=32
- joint right_hip_yaw_joint: limit lower=-2.7576 upper=2.7576 effort=88 velocity=32 -> lower=-2.7576 upper=2.7576 effort=200 velocity=32
- joint right_knee_joint: limit lower=-0.087267 upper=2.8798 effort=139 velocity=20 -> lower=-0.087267 upper=2.8798 effort=250 velocity=20

File: humanoid-legged-description/urdf/humanoid_legged_origin.urdf (robot description, URDF)
Before this commit: robot g1_description, 32 links, 31 joints
Links:
- added link pelvis_contour_link; visual mesh filename=package://humanoid_legged_description/meshes/pelvis_contour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
- added link waist_support_link; visual mesh filename=package://humanoid_legged_description/meshes/waist_support_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
- link left_elbow_link: geometry visual mesh filename=package://humanoid_legged_description/meshes/left_elbow_lin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
- link left_rubber_hand: geometry visual mesh filename=package://humanoid_legged_description/meshes/left_rubber_ha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
- link left_shoulder_pitch_link: geometry visual mesh filename=package://humanoid_legged_description/meshes/left_shoulder_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
- link left_shoulder_roll_link: geometry visual mesh filename=package://humanoid_legged_description/meshes/left_shoulder_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
- link left_shoulder_yaw_link: geometry visual mesh filename=package://humanoid_legged_description/meshes/left_shoulder_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
- link right_elbow_link: geometry visual mesh filename=package://humanoid_legged_description/meshes/right_elbow_li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
- link right_rubber_hand: geometry visual mesh filename=package://humanoid_legged_description/meshes/right_rubber_h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
- link right_shoulder_pitch_link: geometry visual mesh filename=package://humanoid_legged_description/meshes/right_shoulder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
- link right_shoulder_roll_link: geometry visual mesh filename=package://humanoid_legged_description/meshes/right_shoulder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
- link right_shoulder_yaw_link: geometry visual mesh filename=package://humanoid_legged_description/meshes/right_shoulder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
- link waist_roll_link: geometry visual mesh filename=package://humanoid_legged_description/meshes/waist_roll_lin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
- link waist_yaw_link: geometry visual mesh filename=package://humanoid_legged_description/meshes/waist_yaw_link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
Joints:
- added joint pelvis_contour_joint: type fixed, parent pelvis, child pelvis_contour_link, origin xyz=0 0 0 rpy=0 0 0
- added joint waist_support_joint: type fixed, parent pelvis, child waist_support_link, origin xyz=0 0 0 rpy=0 0 0
- joint head_joint: origin xyz=0.0039635 0 0.30 rpy=0 0 0 -> xyz=0.0039635 0 -0.044 rpy=0 0 0
- joint left_shoulder_pitch_joint: origin xyz=0.0039563 0.10022 0.23778 rpy=0 -0.2787 0 -> xyz=0.0039563 0.10022 0.24778 rpy=0.27931 0.000054949 -0.00019159
- joint left_shoulder_roll_joint: origin xyz=0 0.038 -0.013831 rpy=0 0 0 -> xyz=0 0.038 -0.013831 rpy=-0.27925 0 0
- joint right_shoulder_pitch_joint: origin xyz=0.0039563 -0.10021 0.23778 rpy=0 -0.2787 0 -> xyz=0.0039563 -0.10021 0.24778 rpy=-0.27931 0.000054949 0.00019159
- joint right_shoulder_roll_joint: origin xyz=0 -0.038 -0.013831 rpy=0 0 0 -> xyz=0 -0.038 -0.013831 rpy=0.27925 0 0

Commit message: chore: save local changes before syncing main

File: humanoid-legged-description/urdf/humanoid_legged_control.urdf (robot description, URDF)
Before this commit: robot g1_description, 32 links, 31 joints
Joints:
- joint head_joint: origin xyz=0.0039635 0 0.30 rpy=0 0 0 -> xyz=0.0039635 0 -0.054 rpy=0 0 0

File: humanoid-legged-description/urdf/humanoid_legged_origin.urdf (robot description, URDF)
Before this commit: robot g1_description, 32 links, 31 joints
Links:
- added link left_wrist_pitch_link; visual mesh filename=package://humanoid_legged_description/meshes/left_wrist_pit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
- added link left_wrist_roll_link; visual mesh filename=package://humanoid_legged_description/meshes/left_wrist_rol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
- added link left_wrist_yaw_link; visual mesh filename=package://humanoid_legged_description/meshes/left_wrist_yaw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
- added link logo_link; visual mesh filename=package://humanoid_legged_description/meshes/logo_link.STL
- added link pelvis_contour_link; visual mesh filename=package://humanoid_legged_description/meshes/pelvis_contour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
- added link right_wrist_pitch_link; visual mesh filename=package://humanoid_legged_description/meshes/right_wrist_pi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
- added link right_wrist_roll_link; visual mesh filename=package://humanoid_legged_description/meshes/right_wrist_ro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
- added link right_wrist_yaw_link; visual mesh filename=package://humanoid_legged_description/meshes/right_wrist_ya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
- added link waist_support_link; visual mesh filename=package://humanoid_legged_description/meshes/waist_support_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
- link left_elbow_link: geometry visual mesh filename=package://humanoid_legged_description/meshes/left_elbow_lin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
- link left_rubber_hand: geometry visual mesh filename=package://humanoid_legged_description/meshes/left_rubber_ha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
- link left_shoulder_pitch_link: geometry visual mesh filename=package://humanoid_legged_description/meshes/left_shoulder_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
- link left_shoulder_roll_link: geometry visual mesh filename=package://humanoid_legged_description/meshes/left_shoulder_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
- link left_shoulder_yaw_link: geometry visual mesh filename=package://humanoid_legged_description/meshes/left_shoulder_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
- link right_elbow_link: geometry visual mesh filename=package://humanoid_legged_description/meshes/right_elbow_li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
- link right_rubber_hand: geometry visual mesh filename=package://humanoid_legged_description/meshes/right_rubber_h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
- link right_shoulder_pitch_link: geometry visual mesh filename=package://humanoid_legged_description/meshes/right_shoulder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
- link right_shoulder_roll_link: geometry visual mesh filename=package://humanoid_legged_description/meshes/right_shoulder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
- link right_shoulder_yaw_link: geometry visual mesh filename=package://humanoid_legged_description/meshes/right_shoulder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
- link waist_roll_link: geometry visual mesh filename=package://humanoid_legged_description/meshes/waist_roll_lin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
- link waist_yaw_link: geometry visual mesh filename=package://humanoid_legged_description/meshes/waist_yaw_link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
Joints:
- added joint left_wrist_pitch_joint: type fixed, parent left_wrist_roll_link, child left_wrist_pitch_link, origin xyz=0.038 0 0 rpy=0 0 0
- added joint left_wrist_roll_joint: type fixed, parent left_elbow_link, child left_wrist_roll_link, origin xyz=0.1 0.00188791 -0.01 rpy=0 0 0
- added joint left_wrist_yaw_joint: type fixed, parent left_wrist_pitch_link, child left_wrist_yaw_link, origin xyz=0.046 0 0 rpy=0 0 0
- added joint logo_joint: type fixed, parent torso_link, child logo_link, origin xyz=0.0039635 0 -0.054 rpy=0 0 0
- added joint pelvis_contour_joint: type fixed, parent pelvis, child pelvis_contour_link, origin xyz=0 0 0 rpy=0 0 0
- added joint right_wrist_pitch_joint: type fixed, parent right_wrist_roll_link, child right_wrist_pitch_link, origin xyz=0.038 0 0 rpy=0 0 0
- added joint right_wrist_roll_joint: type fixed, parent right_elbow_link, child right_wrist_roll_link, origin xyz=0.1 -0.00188791 -0.01 rpy=0 0 0
- added joint right_wrist_yaw_joint: type fixed, parent right_wrist_pitch_link, child right_wrist_yaw_link, origin xyz=0.046 0 0 rpy=0 0 0
- added joint waist_support_joint: type fixed, parent torso_link, child waist_support_link, origin xyz=0.0039635 0 -0.054 rpy=0 0 0
- joint head_joint: origin xyz=0.0039635 0 0.30 rpy=0 0 0 -> xyz=0.0039635 0 -0.054 rpy=0 0 0
- joint left_hand_joint: origin xyz=0.1 0.00188791 -0.01 rpy=0 0 0 -> xyz=0.0415 0.003 0 rpy=0 0 0; parent left_elbow_link -> left_wrist_yaw_link
- joint right_hand_joint: origin xyz=0.1 -0.00188791 -0.01 rpy=0 0 0 -> xyz=0.0415 -0.003 0 rpy=0 0 0; parent right_elbow_link -> right_wrist_yaw_link

Commit message: Update humanoid controller, gait interface, and simulation sources

File: humanoid-legged-description/urdf/humanoid_legged_control.urdf (robot description, URDF)
Before this commit: robot g1_description, 32 links, 31 joints
Joints:
- joint l_foot_heel_joint: origin xyz=-0.05 0 -0.03 rpy=0 0 0 -> xyz=-0.05 0 -0.035 rpy=0 0 0
- joint l_foot_toe_joint: origin xyz=0.12 0 -0.03 rpy=0 0 0 -> xyz=0.12 0 -0.035 rpy=0 0 0
- joint r_foot_heel_joint: origin xyz=-0.05 0 -0.03 rpy=0 0 0 -> xyz=-0.05 0 -0.035 rpy=0 0 0
- joint r_foot_toe_joint: origin xyz=0.12 0 -0.03 rpy=0 0 0 -> xyz=0.12 0 -0.035 rpy=0 0 0
