Commit message: change to G1 but still has model issue

File: humanoid-legged-description/urdf/humanoid_legged_control.urdf (robot description, URDF)
Before this commit: robot humanoid-legged-description, 32 links, 31 joints
Links:
- removed link arm_l1_link
- removed link arm_l2_link
- removed link arm_l3_link
- removed link arm_l4_link
- removed link arm_l5_link
- removed link arm_l6_link
- removed link arm_r1_link
- removed link arm_r2_link
- removed link arm_r3_link
- removed link arm_r4_link
- removed link arm_r5_link
- removed link arm_r6_link
- removed link base_link
- removed link head_yaw_link
- removed link leg_l1_link
- removed link leg_l2_link
- removed link leg_l3_link
- removed link leg_l4_link
- removed link leg_l5_link
- removed link leg_l6_link
- removed link leg_r1_link
- removed link leg_r2_link
- removed link leg_r3_link
- removed link leg_r4_link
- removed link leg_r5_link
- removed link leg_r6_link
- added link head_link, mass 1.036
- added link left_ankle_pitch_link, mass 0.074
- added link left_ankle_roll_link, mass 0.608; collision box size=0.18 0.08 0.01
- added link left_elbow_link, mass 0.6
- added link left_hip_pitch_link, mass 1.35
- added link left_hip_roll_link, mass 1.52
- added link left_hip_yaw_link, mass 1.702
- added link left_knee_link, mass 1.932
- added link left_rubber_hand, mass 0.824
- added link left_shoulder_pitch_link, mass 0.718
- added link left_shoulder_roll_link, mass 0.643
- added link left_shoulder_yaw_link, mass 0.734
- added link pelvis, mass 3.813; collision box size=0.15 0.2 0.15
- added link right_ankle_pitch_link, mass 0.074
- added link right_ankle_roll_link, mass 0.608; collision box size=0.18 0.08 0.01
- added link right_elbow_link, mass 0.6
- added link right_hip_pitch_link, mass 1.35
- added link right_hip_roll_link, mass 1.52
- added link right_hip_yaw_link, mass 1.702
- added link right_knee_link, mass 1.932
- added link right_rubber_hand, mass 0.824
- added link right_shoulder_pitch_link, mass 0.718
- added link right_shoulder_roll_link, mass 0.643
- added link right_shoulder_yaw_link, mass 0.734
- added link torso_link, mass 9.598; collision box size=0.2 0.3 0.35
- added link waist_roll_link, mass 0.047
- link waist_yaw_link: mass 8.000000 -> 0.244; geometry 
Joints:
- removed joint arm_l1_joint
- removed joint arm_l2_joint
- removed joint arm_l3_joint
- removed joint arm_l4_joint
- removed joint arm_l5_joint
- removed joint arm_l6_joint
- removed joint arm_r1_joint
- removed joint arm_r2_joint
- removed joint arm_r3_joint
- removed joint arm_r4_joint
- removed joint arm_r5_joint
- removed joint arm_r6_joint
- removed joint dummy_to_base_link
- removed joint head_yaw_joint
- removed joint leg_l1_joint
- removed joint leg_l2_joint
- removed joint leg_l3_joint
- removed joint leg_l4_joint
- removed joint leg_l5_joint
- removed joint leg_l6_joint
- removed joint leg_r1_joint
- removed joint leg_r2_joint
- removed joint leg_r3_joint
- removed joint leg_r4_joint
- removed joint leg_r5_joint
- removed joint leg_r6_joint
- added joint dummy_to_pelvis: type fixed, parent dummy_link, child pelvis, origin xyz=0 0 0 rpy=0 0 0
- added joint head_joint: type fixed, parent torso_link, child head_link, origin xyz=0.0039635 0 -0.044 rpy=0 0 0
- added joint left_ankle_pitch_joint: type revolute, parent left_knee_link, child left_ankle_pitch_link, origin xyz=0 -9.4445e-05 -0.30001 rpy=0 0 0, axis 0 1 0, limit lower=-0.87267 upper=0.5236 effort=120 velocity=30
- added joint left_ankle_roll_joint: type revolute, parent left_ankle_pitch_link, child left_ankle_roll_link, origin xyz=0 0 -0.017558 rpy=0 0 0, axis 1 0 0, limit lower=-0.2618 upper=0.2618 effort=120 velocity=30
- added joint left_elbow_joint: type fixed, parent left_shoulder_yaw_link, child left_elbow_link, origin xyz=0.015783 0 -0.080518 rpy=0 0 0
- added joint left_hand_joint: type fixed, parent left_elbow_link, child left_rubber_hand, origin xyz=0.1 0.00188791 -0.01 rpy=0 0 0
- added joint left_hip_pitch_joint: type revolute, parent pelvis, child left_hip_pitch_link, origin xyz=0 0.064452 -0.1027 rpy=0 0 0, axis 0 1 0, limit lower=-2.5307 upper=2.8798 effort=200 velocity=32
- added joint left_hip_roll_joint: type revolute, parent left_hip_pitch_link, child left_hip_roll_link, origin xyz=0 0.052 -0.030465 rpy=0 -0.1749 0, axis 1 0 0, limit lower=-0.5236 upper=2.9671 effort=200 velocity=32
- added joint left_hip_yaw_joint: type revolute, parent left_hip_roll_link, child left_hip_yaw_link, origin xyz=0.025001 0 -0.12412 rpy=0 0 0, axis 0 0 1, limit lower=-2.7576 upper=2.7576 effort=200 velocity=32
- added joint left_knee_joint: type revolute, parent left_hip_yaw_link, child left_knee_link, origin xyz=-0.078273 0.0021489 -0.17734 rpy=0 0.1749 0, axis 0 1 0, limit lower=-0.087267 upper=2.8798 effort=250 velocity=20
- added joint left_shoulder_pitch_joint: type fixed, parent torso_link, child left_shoulder_pitch_link, origin xyz=0.0039563 0.10022 0.23778 rpy=0 -0.2787 0
- added joint left_shoulder_roll_joint: type fixed, parent left_shoulder_pitch_link, child left_shoulder_roll_link, origin xyz=0 0.038 -0.013831 rpy=0 0 0
- added joint left_shoulder_yaw_joint: type fixed, parent left_shoulder_roll_link, child left_shoulder_yaw_link, origin xyz=0 0.00624 -0.1032 rpy=0 0 0
- added joint right_ankle_pitch_joint: type revolute, parent right_knee_link, child right_ankle_pitch_link, origin xyz=0 9.4445e-05 -0.30001 rpy=0 0 0, axis 0 1 0, limit lower=-0.87267 upper=0.5236 effort=120 velocity=30
- added joint right_ankle_roll_joint: type revolute, parent right_ankle_pitch_link, child right_ankle_roll_link, origin xyz=0 0 -0.017558 rpy=0 0 0, axis 1 0 0, limit lower=-0.2618 upper=0.2618 effort=120 velocity=30
- added joint right_elbow_joint: type fixed, parent right_shoulder_yaw_link, child right_elbow_link, origin xyz=0.015783 0 -0.080518 rpy=0 0 0
- added joint right_hand_joint: type fixed, parent right_elbow_link, child right_rubber_hand, origin xyz=0.1 -0.00188791 -0.01 rpy=0 0 0
- added joint right_hip_pitch_joint: type revolute, parent pelvis, child right_hip_pitch_link, origin xyz=0 -0.064452 -0.1027 rpy=0 0 0, axis 0 1 0, limit lower=-2.5307 upper=2.8798 effort=200 velocity=32
- added joint right_hip_roll_joint: type revolute, parent right_hip_pitch_link, child right_hip_roll_link, origin xyz=0 -0.052 -0.030465 rpy=0 -0.1749 0, axis 1 0 0, limit lower=-2.9671 upper=0.5236 effort=200 velocity=32
- added joint right_hip_yaw_joint: type revolute, parent right_hip_roll_link, child right_hip_yaw_link, origin xyz=0.025001 0 -0.12412 rpy=0 0 0, axis 0 0 1, limit lower=-2.7576 upper=2.7576 effort=200 velocity=32
- added joint right_knee_joint: type revolute, parent right_hip_yaw_link, child right_knee_link, origin xyz=-0.078273 -0.0021489 -0.17734 rpy=0 0.1749 0, axis 0 1 0, limit lower=-0.087267 upper=2.8798 effort=250 velocity=20
- added joint right_shoulder_pitch_joint: type fixed, parent torso_link, child right_shoulder_pitch_link, origin xyz=0.0039563 -0.10021 0.23778 rpy=0 -0.2787 0
- added joint right_shoulder_roll_joint: type fixed, parent right_shoulder_pitch_link, child right_shoulder_roll_link, origin xyz=0 -0.038 -0.013831 rpy=0 0 0
- added joint right_shoulder_yaw_joint: type fixed, parent right_shoulder_roll_link, child right_shoulder_yaw_link, origin xyz=0 -0.00624 -0.1032 rpy=0 0 0
- added joint waist_pitch_joint: type fixed, parent waist_roll_link, child torso_link, origin xyz=0 0 0.019 rpy=0 0 0
- added joint waist_roll_joint: type fixed, parent waist_yaw_link, child waist_roll_link, origin xyz=-0.0039635 0 0.035 rpy=0 0 0
- joint l_foot_heel_joint: origin xyz=0 -0.033 -0.0445 rpy=0 0 0 -> xyz=-0.05 0 -0.035 rpy=0 0 0; parent leg_l6_link -> left_ankle_roll_link
- joint l_foot_toe_joint: origin xyz=0 -0.033 0.1415 rpy=0 0 0 -> xyz=0.12 0 -0.035 rpy=0 0 0; parent leg_l6_link -> left_ankle_roll_link
- joint r_foot_heel_joint: origin xyz=0 -0.033 -0.0445 rpy=0 0 0 -> xyz=-0.05 0 -0.035 rpy=0 0 0; parent leg_r6_link -> right_ankle_roll_link
- joint r_foot_toe_joint: origin xyz=0 -0.033 0.1415 rpy=0 0 0 -> xyz=0.12 0 -0.035 rpy=0 0 0; parent leg_r6_link -> right_ankle_roll_link
- joint waist_yaw_joint: axis 0 0 1 -> (none); limit lower=-1.5708 upper=1.5708 effort=150.0 velocity=12.0 -> (none); origin xyz=0 0 -0.24015 rpy=0 0 0 -> xyz=0 0 0 rpy=0 0 0; parent base_link -> pelvis

File: humanoid-legged-description/urdf/humanoid_legged_origin.urdf (robot description, URDF)
Before this commit: robot humanoid_legged_description, 32 links, 31 joints
Links:
- removed link arm_l1_link
- removed link arm_l2_link
- removed link arm_l3_link
- removed link arm_l4_link
- removed link arm_l5_link
- removed link arm_l6_link
- removed link arm_r1_link
- removed link arm_r2_link
- removed link arm_r3_link
- removed link arm_r4_link
- removed link arm_r5_link
- removed link arm_r6_link
- removed link base_link
- removed link head_yaw_link
- removed link leg_l1_link
- removed link leg_l2_link
- removed link leg_l3_link
- removed link leg_l4_link
- removed link leg_l5_link
- removed link leg_l6_link
- removed link leg_r1_link
- removed link leg_r2_link
- removed link leg_r3_link
- removed link leg_r4_link
- removed link leg_r5_link
- removed link leg_r6_link
- added link head_link, mass 1.036; visual mesh filename=package://humanoid_legged_description/meshes/head_link.STL
- added link left_ankle_pitch_link, mass 0.074; visual mesh filename=package://humanoid_legged_description/meshes/left_ankle_pit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
- added link left_ankle_roll_link, mass 0.608; collision box size=0.18 0.08 0.01; visual mesh filename=package://humanoid_legged_description/meshes/left_ankle_rol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
- added link left_elbow_link, mass 0.6; visual mesh filename=package://humanoid_legged_description/meshes/left_elbow_lin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
- added link left_hip_pitch_link, mass 1.35; visual mesh filename=package://humanoid_legged_description/meshes/left_hip_pitch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
- added link left_hip_roll_link, mass 1.52; visual mesh filename=package://humanoid_legged_description/meshes/left_hip_roll_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
- added link left_hip_yaw_link, mass 1.702; visual mesh filename=package://humanoid_legged_description/meshes/left_hip_yaw_l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
- added link left_knee_link, mass 1.932; visual mesh filename=package://humanoid_legged_description/meshes/left_knee_link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
- added link left_rubber_hand, mass 0.824; visual mesh filename=package://humanoid_legged_description/meshes/left_rubber_ha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
- added link left_shoulder_pitch_link, mass 0.718; visual mesh filename=package://humanoid_legged_description/meshes/left_shoulder_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
- added link left_shoulder_roll_link, mass 0.643; visual mesh filename=package://humanoid_legged_description/meshes/left_shoulder_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
- added link left_shoulder_yaw_link, mass 0.734; visual mesh filename=package://humanoid_legged_description/meshes/left_shoulder_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
- added link pelvis, mass 3.813; collision box size=0.15 0.2 0.15; visual mesh filename=package://humanoid_legged_description/meshes/pelvis.STL
- added link pelvis_contour_link; visual mesh filename=package://humanoid_legged_description/meshes/pelvis_contour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
- added link right_ankle_pitch_link, mass 0.074; visual mesh filename=package://humanoid_legged_description/meshes/right_ankle_pi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
- added link right_ankle_roll_link, mass 0.608; collision box size=0.18 0.08 0.01; visual mesh filename=package://humanoid_legged_description/meshes/right_ankle_ro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
- added link right_elbow_link, mass 0.6; visual mesh filename=package://humanoid_legged_description/meshes/right_elbow_li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
- added link right_hip_pitch_link, mass 1.35; visual mesh filename=package://humanoid_legged_description/meshes/right_hip_pitc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
- added link right_hip_roll_link, mass 1.52; visual mesh filename=package://humanoid_legged_description/meshes/right_hip_roll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
- added link right_hip_yaw_link, mass 1.702; visual mesh filename=package://humanoid_legged_description/meshes/right_hip_yaw_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
- added link right_knee_link, mass 1.932; visual mesh filename=package://humanoid_legged_description/meshes/right_knee_lin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
- added link right_rubber_hand, mass 0.824; visual mesh filename=package://humanoid_legged_description/meshes/right_rubber_h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
- added link right_shoulder_pitch_link, mass 0.718; visual mesh filename=package://humanoid_legged_description/meshes/right_shoulder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
- added link right_shoulder_roll_link, mass 0.643; visual mesh filename=package://humanoid_legged_description/meshes/right_shoulder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
- added link right_shoulder_yaw_link, mass 0.734; visual mesh filename=package://humanoid_legged_description/meshes/right_shoulder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
- added link torso_link, mass 9.598; collision box size=0.2 0.3 0.35; visual mesh filename=package://humanoid_legged_description/meshes/torso_link.STL
- added link waist_roll_link, mass 0.047; visual mesh filename=package://humanoid_legged_description/meshes/waist_roll_lin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
- added link waist_support_link; visual mesh filename=package://humanoid_legged_description/meshes/waist_support_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
- link waist_yaw_link: mass 8.000000 -> 0.244; geometry visual mesh filename=package://humanoid_legged_description/meshes/waist_yaw_link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
Joints:
- removed joint arm_l1_joint
- removed joint arm_l2_joint
- removed joint arm_l3_joint
- removed joint arm_l4_joint
- removed joint arm_l5_joint
- removed joint arm_l6_joint
- removed joint arm_r1_joint
- removed joint arm_r2_joint
- removed joint arm_r3_joint
- removed joint arm_r4_joint
- removed joint arm_r5_joint
- removed joint arm_r6_joint
- removed joint dummy_to_base_link
- removed joint head_yaw_joint
- removed joint leg_l1_joint
- removed joint leg_l2_joint
- removed joint leg_l3_joint
- removed joint leg_l4_joint
- removed joint leg_l5_joint
- removed joint leg_l6_joint
- removed joint leg_r1_joint
- removed joint leg_r2_joint
- removed joint leg_r3_joint
- removed joint leg_r4_joint
- removed joint leg_r5_joint
- removed joint leg_r6_joint
- added joint dummy_to_pelvis: type fixed, parent dummy_link, child pelvis, origin xyz=0 0 0 rpy=0 0 0
- added joint head_joint: type fixed, parent torso_link, child head_link, origin xyz=0.0039635 0 -0.044 rpy=0 0 0
- added joint left_ankle_pitch_joint: type revolute, parent left_knee_link, child left_ankle_pitch_link, origin xyz=0 -9.4445e-05 -0.30001 rpy=0 0 0, axis 0 1 0, limit lower=-0.87267 upper=0.5236 effort=50 velocity=30
- added joint left_ankle_roll_joint: type revolute, parent left_ankle_pitch_link, child left_ankle_roll_link, origin xyz=0 0 -0.017558 rpy=0 0 0, axis 1 0 0, limit lower=-0.2618 upper=0.2618 effort=50 velocity=30
- added joint left_elbow_joint: type fixed, parent left_shoulder_yaw_link, child left_elbow_link, origin xyz=0.015783 0 -0.080518 rpy=0 0 0
- added joint left_hand_joint: type fixed, parent left_elbow_link, child left_rubber_hand, origin xyz=0.1 0.00188791 -0.01 rpy=0 0 0
- added joint left_hip_pitch_joint: type revolute, parent pelvis, child left_hip_pitch_link, origin xyz=0 0.064452 -0.1027 rpy=0 0 0, axis 0 1 0, limit lower=-2.5307 upper=2.8798 effort=88 velocity=32
- added joint left_hip_roll_joint: type revolute, parent left_hip_pitch_link, child left_hip_roll_link, origin xyz=0 0.052 -0.030465 rpy=0 -0.1749 0, axis 1 0 0, limit lower=-0.5236 upper=2.9671 effort=88 velocity=32
- added joint left_hip_yaw_joint: type revolute, parent left_hip_roll_link, child left_hip_yaw_link, origin xyz=0.025001 0 -0.12412 rpy=0 0 0, axis 0 0 1, limit lower=-2.7576 upper=2.7576 effort=88 velocity=32
- added joint left_knee_joint: type revolute, parent left_hip_yaw_link, child left_knee_link, origin xyz=-0.078273 0.0021489 -0.17734 rpy=0 0.1749 0, axis 0 1 0, limit lower=-0.087267 upper=2.8798 effort=139 velocity=20
- added joint left_shoulder_pitch_joint: type fixed, parent torso_link, child left_shoulder_pitch_link, origin xyz=0.0039563 0.10022 0.24778 rpy=0.27931 0.000054949 -0.00019159
- added joint left_shoulder_roll_joint: type fixed, parent left_shoulder_pitch_link, child left_shoulder_roll_link, origin xyz=0 0.038 -0.013831 rpy=-0.27925 0 0
- added joint left_shoulder_yaw_joint: type fixed, parent left_shoulder_roll_link, child left_shoulder_yaw_link, origin xyz=0 0.00624 -0.1032 rpy=0 0 0
- added joint pelvis_contour_joint: type fixed, parent pelvis, child pelvis_contour_link, origin xyz=0 0 0 rpy=0 0 0
- added joint right_ankle_pitch_joint: type revolute, parent right_knee_link, child right_ankle_pitch_link, origin xyz=0 9.4445e-05 -0.30001 rpy=0 0 0, axis 0 1 0, limit lower=-0.87267 upper=0.5236 effort=50 velocity=30
- added joint right_ankle_roll_joint: type revolute, parent right_ankle_pitch_link, child right_ankle_roll_link, origin xyz=0 0 -0.017558 rpy=0 0 0, axis 1 0 0, limit lower=-0.2618 upper=0.2618 effort=50 velocity=30
- added joint right_elbow_joint: type fixed, parent right_shoulder_yaw_link, child right_elbow_link, origin xyz=0.015783 0 -0.080518 rpy=0 0 0
- added joint right_hand_joint: type fixed, parent right_elbow_link, child right_rubber_hand, origin xyz=0.1 -0.00188791 -0.01 rpy=0 0 0
- added joint right_hip_pitch_joint: type revolute, parent pelvis, child right_hip_pitch_link, origin xyz=0 -0.064452 -0.1027 rpy=0 0 0, axis 0 1 0, limit lower=-2.5307 upper=2.8798 effort=88 velocity=32
- added joint right_hip_roll_joint: type revolute, parent right_hip_pitch_link, child right_hip_roll_link, origin xyz=0 -0.052 -0.030465 rpy=0 -0.1749 0, axis 1 0 0, limit lower=-2.9671 upper=0.5236 effort=88 velocity=32
- added joint right_hip_yaw_joint: type revolute, parent right_hip_roll_link, child right_hip_yaw_link, origin xyz=0.025001 0 -0.12412 rpy=0 0 0, axis 0 0 1, limit lower=-2.7576 upper=2.7576 effort=88 velocity=32
- added joint right_knee_joint: type revolute, parent right_hip_yaw_link, child right_knee_link, origin xyz=-0.078273 -0.0021489 -0.17734 rpy=0 0.1749 0, axis 0 1 0, limit lower=-0.087267 upper=2.8798 effort=139 velocity=20
- added joint right_shoulder_pitch_joint: type fixed, parent torso_link, child right_shoulder_pitch_link, origin xyz=0.0039563 -0.10021 0.24778 rpy=-0.27931 0.000054949 0.00019159
- added joint right_shoulder_roll_joint: type fixed, parent right_shoulder_pitch_link, child right_shoulder_roll_link, origin xyz=0 -0.038 -0.013831 rpy=0.27925 0 0
- added joint right_shoulder_yaw_joint: type fixed, parent right_shoulder_roll_link, child right_shoulder_yaw_link, origin xyz=0 -0.00624 -0.1032 rpy=0 0 0
- added joint waist_pitch_joint: type fixed, parent waist_roll_link, child torso_link, origin xyz=0 0 0.019 rpy=0 0 0
- added joint waist_roll_joint: type fixed, parent waist_yaw_link, child waist_roll_link, origin xyz=-0.0039635 0 0.035 rpy=0 0 0
- added joint waist_support_joint: type fixed, parent pelvis, child waist_support_link, origin xyz=0 0 0 rpy=0 0 0
- joint l_foot_heel_joint: origin xyz=0 -0.033 -0.0445 rpy=0 0 0 -> xyz=-0.05 0 -0.03 rpy=0 0 0; parent leg_l6_link -> left_ankle_roll_link
- joint l_foot_toe_joint: origin xyz=0 -0.033 0.1415 rpy=0 0 0 -> xyz=0.12 0 -0.03 rpy=0 0 0; parent leg_l6_link -> left_ankle_roll_link
- joint r_foot_heel_joint: origin xyz=0 -0.033 -0.0445 rpy=0 0 0 -> xyz=-0.05 0 -0.03 rpy=0 0 0; parent leg_r6_link -> right_ankle_roll_link
- joint r_foot_toe_joint: origin xyz=0 -0.033 0.1415 rpy=0 0 0 -> xyz=0.12 0 -0.03 rpy=0 0 0; parent leg_r6_link -> right_ankle_roll_link
- joint waist_yaw_joint: axis 0 0 1 -> (none); limit lower=-1.5708 upper=1.5708 effort=150.0 velocity=12.0 -> (none); origin xyz=0 0 -0.24015 rpy=0 0 0 -> xyz=0 0 0 rpy=0 0 0; parent base_link -> pelvis
